File: PHAT-3 Main Board.kicad_sch (KiCad schematic)
At the start: 30 parts, among them P1 Power Terminal Block, P2 Power Terminal Block, P3 Power Terminal Block, P4 Power Terminal Block, Q1 IRLZ44N, SW2 SW_DPDT_x2, U1 AHT21, U10 Logic Level Converter, U2 ESP32-S3 Dual-core SX1262, U3 GY-68 BMP180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

Commit message: Final touches! :)
Connections:
- net +15V: now also SW2.2 (B); no longer P1.2 (PWR)
- net GND: now also C4.2, D1.2 (A), U5.3 (IN-); no longer D1.1 (K), SW2.2 (B)
- net at P1.1 (GND): now also D1.1 (K); no longer SW2.1 (A)
- new net: P1.2 (PWR), SW2.1 (A)
Other:
- moved on the sheet: D1, SW2A
