File: PHAT-3 Main Board.kicad_pcb (KiCad board)
At the start: 6 copper layers, 95.9 x 90.2 mm, 34 parts, among them P1 Power Terminal Block, P2 Power Terminal Block, P3 Power Terminal Block, P4 Power Terminal Block, Q1 IRLZ44N, SW2 SW_DPDT_x2, U1 AHT21, U10 Logic Level Converter, U2 ESP32-S3 Dual-core SX1262, U3 GY-68 BMP180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

Commit message: Routed the PCB.
Parts:
- moved C4 1.51 mm to (173.0, 61.5), turned to 0 degrees
Routing:
- net Net-(U1-SCL): track 0.00 -> 137.8 mm
- net Net-(U1-SDA): track 0.00 -> 129.3 mm
- net +15V: track 0.00 -> 56.9 mm
- net Net-(U2-U1TXD): track 0.00 -> 36.8 mm
- net Net-(U2-MISO): track 0.00 -> 36.5 mm
- net Net-(U2-U2RXD): track 0.00 -> 36.0 mm
- net Net-(U2-U1RXD): track 0.00 -> 34.7 mm
- net Net-(D1-A): track 0.00 -> 34.5 mm
- net Net-(U2-U2TXD): track 0.00 -> 33.9 mm
- net Net-(D2-A): track 0.00 -> 30.8 mm
- net Net-(U2-HTR): track 0.00 -> 26.7 mm
- net Net-(U10-HV2): track 0.00 -> 23.7 mm
- net Net-(U10-HV1): track 0.00 -> 23.3 mm
- net Net-(U2-CS): track 0.00 -> 19.6 mm
- net Net-(D3-A): track 0.00 -> 17.2 mm
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- added copper zone on In3.Cu, net +3V3
- added copper zone on In2.Cu, net +5V
- added copper zone on In1.Cu, net GND

Commit message: Final touches! :)
Parts:
- REF** (x4): value MountingHole_3.2mm_M3 -> MountingHole_3.2mm_M3_Pad_Via; footprint MountingHole:MountingHole_3.2mm_M3 -> MountingHole:MountingHole_3.2mm_M3_Pad_Via
- moved D1 13.0 mm to (181.7, 59.5), turned to -90 degrees
Connections:
- C4 pad 2: Net-(D1-A) -> GND
- D1 pad 1: GND -> Net-(D1-K)
- D1 pad 2: Net-(D1-A) -> GND
- P1 pad 1: Net-(P1-GND) -> Net-(D1-K)
- P1 pad 2: +15V -> Net-(P1-PWR)
- SW2 pad 1: Net-(P1-GND) -> Net-(P1-PWR)
- SW2 pad 2: GND -> +15V
- U5 pad 3: Net-(D1-A) -> GND
Routing:
- net Net-(D1-A): track 34.5 -> 0.00 mm
- net Net-(P1-PWR): track 0.00 -> 21.8 mm
- net Net-(P1-GND): track 15.6 -> 0.00 mm
- net Net-(D1-K): track 0.00 -> 8.52 mm
- net +15V: track 56.9 -> 52.1 mm
Other:
- board text added: "+15V"
- board text added: "+5V"
- board text added: "GND"

Commit message: Final revision FINAL_FINAL_2
Other:
- board text added: "Designed by Yehoshua Luna with kind help from Marcin Anforowicz, Evan Gubarev, Shriya Tiku, and David Magidson. Feb. 2025 https://github.com/UWCubeSat/PHAT-3-Main-Board"
- board text added: "PHAT-3"
- board text removed: "Designed by Yehoshua Luna with kind help from Marcin Anforowicz and Evan Gubarev. https://github.com/UWCubeSat/PHAT-3-Main-Board"
Changed lines of the file:
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@@
+		)
+	)
+	(gr_text "PHAT-3"
+		(at 109 118 -90)
+		(layer "B.SilkS" knockout)
+		(effects
+			(font
+				(size 10 10)
+				(thickness 2.5)
+				(bold yes)
+			)
+			(justify left bottom mirror)
 		)
 	)
@@
 		)
 	)
-	(gr_text "Designed by Yehoshua Luna with kind help from Marcin Anforowicz and Evan Gubarev.\n\nhttps://github.com/UWCubeSat/PHAT-3-Main-Board"
-		(at 143.383 93.299 -90)
+	(gr_text "Designed by Yehoshua Luna with kind help from Marcin Anforowicz,\nEvan Gubarev, Shriya Tiku, and David Magidson.\n\nFeb. 2025\n\nhttps://github.com/UWCubeSat/PHAT-3-Main-Board"
+		(at 139.5 93.5 270)
 		(layer "B.SilkS")
 		(effects
